File: Player!.kicad_sch (KiCad schematic)
At the start: 25 parts, among them J1 USB4085-GF-A_REVA4, SW1 RotaryEncoder_Switch, SW2 SW_Push, SW3 SW_Push, SW4 SW_Push, SW5 SW_Push, U1 ATmega328P-P, Y1 Crystal

Commit message: Minor text changes
Parts:
- renumbered U1 to ATMega328, BOOT1 to Boot, Y1 to Crystal, LED1 to Power, RESET1 to Reset
Changed lines of the file:
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@@
   (symbol (lib_id "MCU_Microchip_ATmega:ATmega328P-P") (at 44.45 166.37 0) (unit 1)
     (in_bom yes) (on_board yes) (fields_autoplaced)
-    (property "Reference" "U1" (id 0) (at 23.4701 132.1648 0))
+    (property "Reference" "ATMega328" (id 0) (at 23.4701 132.1648 0))
     (property "Value" "ATmega328P-P" (id 1) (at 23.4701 134.9399 0))
     (property "Footprint" "Keyboard Stuff:ATmega328p DIP-28" (id 2) (at 44.45 166.37 0)
@@
   (symbol (lib_id "Device:Crystal_Small") (at 77.47 153.67 0) (unit 1)
     (in_bom yes) (on_board yes)
-    (property "Reference" "Y1" (id 0) (at 76.2 149.86 0)
+    (property "Reference" "Crystal" (id 0) (at 76.2 149.86 0)
       (effects (font (size 1.27 1.27)) (justify left))
     )
@@
   (symbol (lib_id "keyboard_parts:SW_PUSH") (at 77.47 191.77 0) (mirror y) (unit 1)
     (in_bom yes) (on_board yes)
-    (property "Reference" "BOOT1" (id 0) (at 77.47 185.293 0))
+    (property "Reference" "Boot" (id 0) (at 77.47 185.293 0))
     (property "Value" "BOOT" (id 1) (at 77.47 187.6044 0))
     (property "Footprint" "Keyboard_Stuff:SW_PUSH_6mm" (id 2) (at 77.47 191.77 0)
@@
   (symbol (lib_id "Device:LED") (at 143.51 207.645 0) (unit 1)
     (in_bom yes) (on_board yes) (fields_autoplaced)
-    (property "Reference" "LED1" (id 0) (at 141.9225 202.4085 0))
+    (property "Reference" "Power" (id 0) (at 141.9225 202.4085 0))
     (property "Value" "POWERLED" (id 1) (at 141.9225 205.1836 0))
     (property "Footprint" "Keyboard_Stuff:LED_D3.0mm" (id 2) (at 143.51 207.645 0)
@@
   (symbol (lib_id "keyboard_parts:SW_PUSH") (at 79.375 173.99 0) (mirror y) (unit 1)
     (in_bom yes) (on_board yes)
-    (property "Reference" "RESET1" (id 0) (at 79.375 167.513 0))
+    (property "Reference" "Reset" (id 0) (at 79.375 167.513 0))
     (property "Value" "RESET" (id 1) (at 79.375 169.8244 0))
     (property "Footprint" "Keyboard_Stuff:SW_PUSH_6mm" (id 2) (at 79.375 173.99 0)
@@
       (reference "#PWR021") (unit 1) (value "+5V") (footprint "")
     )
+    (path "/16753c81-1a3b-47e2-8a5b-29fa84e3a60a"
+      (reference "ATMega328") (unit 1) (value "ATmega328P-P") (footprint "Keyboard Stuff:ATmega328p DIP-28")
+    )
     (path "/49339521-16b8-463d-be4d-2afce06e238b"
-      (reference "BOOT1") (unit 1) (value "BOOT") (footprint "Keyboard_Stuff:SW_PUSH_6mm")
+      (reference "Boot") (unit 1) (value "BOOT") (footprint "Keyboard_Stuff:SW_PUSH_6mm")
     )
     (path "/8a43a549-7c53-4159-9079-e3706117cb9f"
@@
       (reference "C5") (unit 1) (value "4.7u") (footprint "Keyboard_Stuff:CP_Radial_D4.0mm_P1.50mm")
     )
+    (path "/28eb2027-6d9a-4962-9497-a4b3a97fc4a9"
+      (reference "Crystal") (unit 1) (value "Crystal") (footprint "Keyboard Stuff:Crystal_HC49-4H_Vertical")
+    )
     (path "/013d12e2-bc18-4c37-b184-538605215685"
       (reference "DN1") (unit 1) (value "3.6V") (footprint "Keyboard_Stuff:D_DO-35_SOD27_P5.08mm_Vertical_AnodeUp")
@@
     )
     (path "/56d3b62a-1ebf-4e13-b8a1-2c403d0824ee"
-      (reference "LED1") (unit 1) (value "POWERLED") (footprint "Keyboard_Stuff:LED_D3.0mm")
+      (reference "Power") (unit 1) (value "POWERLED") (footprint "Keyboard_Stuff:LED_D3.0mm")
     )
     (path "/eaf0749f-fc67-4f3c-9a2d-cfa1273640a6"
@@
     )
     (path "/6d8c26be-6a42-402b-acee-7b1a9d70afbd"
-      (reference "RESET1") (unit 1) (value "RESET") (footprint "Keyboard_Stuff:SW_PUSH_6mm")
+      (reference "Reset") (unit 1) (value "RESET") (footprint "Keyboard_Stuff:SW_PUSH_6mm")
     )
     (path "/7752d938-57d5-41f4-96c4-d071fa08efc1"
@@
       (reference "SW5") (unit 1) (value "SW_Push") (footprint "Keyboard Stuff:Player! 1u PCB")
     )
-    (path "/16753c81-1a3b-47e2-8a5b-29fa84e3a60a"
-      (reference "U1") (unit 1) (value "ATmega328P-P") (footprint "Keyboard Stuff:ATmega328p DIP-28")
-    )
-    (path "/28eb2027-6d9a-4962-9497-a4b3a97fc4a9"
-      (reference "Y1") (unit 1) (value "Crystal") (footprint "Keyboard Stuff:Crystal_HC49-4H_Vertical")
-    )
-  )
+  )

Commit message: Update PCB
Updated the PCB to include new models for rotary encoder with cap, cherry keys with keycaps. Also reordered some components and added a new horizontal zener diode model
Parts:
- DN1: footprint Keyboard_Stuff:D_DO-35_SOD27_P5.08mm_Vertical_AnodeUp -> Keyboard_Stuff:D_DO-35_SOD27_P5.08mm_Horizontal
- DP1: footprint Keyboard_Stuff:D_DO-35_SOD27_P5.08mm_Vertical_AnodeUp -> Keyboard Stuff:D_DO-35_SOD27_P5.08mm_Horizontal
- renumbered Boot to Boot1, Crystal to Crystal1, Power to Power1, Reset to Reset1, SW5 to SW1, SW1 to SW5
Connections:
- net GND: now also R7.2; no longer R7.1
- net LED: now also R7.1; no longer R7.2
- net SW1: now also SW1.1; no longer SW5.S2
- net SW5: now also SW5.S2; no longer SW1.1
Other:
- moved on the sheet: R7, SW1, SW2, SW3, SW4
