File: Player!.kicad_sch (KiCad schematic)
At the start: 25 parts, among them J1 USB4085-GF-A_REVA4, SW1 SW_Push, SW2 SW_Push, SW3 SW_Push, SW4 SW_Push, SW5 RotaryEncoder_Switch

Commit message: Updated Models
Changed type C footprint & model, updated to use .step models in 3d for all components
Parts:
- J1: footprint Keyboard Stuff:USB_C_Receptacle_GCT_USB4085 -> Keyboard Stuff:GCT_USB4085-GF-A_REVA4
Changed lines of the file:
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@@
     (property "Reference" "J1" (id 0) (at 36.83 219.5535 0))
     (property "Value" "USB4085-GF-A_REVA4" (id 1) (at 36.83 222.3286 0))
-    (property "Footprint" "Keyboard Stuff:USB_C_Receptacle_GCT_USB4085" (id 2) (at 36.83 241.3 0)
+    (property "Footprint" "Keyboard Stuff:GCT_USB4085-GF-A_REVA4" (id 2) (at 36.83 241.3 0)
       (effects (font (size 1.27 1.27)) (justify left bottom) hide)
     )
@@
     )
     (path "/315cc8b8-91a5-48ab-9789-390f34a7043c"
-      (reference "J1") (unit 1) (value "USB4085-GF-A_REVA4") (footprint "Keyboard Stuff:USB_C_Receptacle_GCT_USB4085")
+      (reference "J1") (unit 1) (value "USB4085-GF-A_REVA4") (footprint "Keyboard Stuff:GCT_USB4085-GF-A_REVA4")
     )
     (path "/56d3b62a-1ebf-4e13-b8a1-2c403d0824ee"

Commit message: Updating PCB and Models for Case
Parts:
- renumbered R7 to R1, R4 to R3, R3 to R4, R1 to R5, R5 to R7
Changed lines of the file:
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@@
   (junction (at 127 149.86) (diameter 0) (color 0 0 0 0)
   )
+  (junction (at 74.93 153.67) (diameter 0) (color 0 0 0 0)
+  )
   (junction (at 100.33 242.57) (diameter 0) (color 0 0 0 0)
   )
@@
   )
   (junction (at 67.31 254) (diameter 0) (color 0 0 0 0)
-  )
-  (junction (at 74.93 153.67) (diameter 0) (color 0 0 0 0)
   )
   (no_connect (at 59.69 135.89))
@@
     (stroke (width 0) (type default) (color 0 0 0 0))
   )
-  (wire (pts (xy 80.01 151.13) (xy 59.69 151.13))
-    (stroke (width 0) (type default) (color 0 0 0 0))
-  )
   (wire (pts (xy 147.32 207.645) (xy 149.86 207.645))
     (stroke (width 0) (type default) (color 0 0 0 0))
@@
     (stroke (width 0) (type default) (color 0 0 0 0))
   )
+  (wire (pts (xy 59.69 153.67) (xy 74.93 153.67))
+    (stroke (width 0) (type default) (color 0 0 0 0))
+  )
   (wire (pts (xy 49.53 223.52) (xy 49.53 256.54))
     (stroke (width 0) (type default) (color 0 0 0 0))
@@
     (stroke (width 0) (type default) (color 0 0 0 0))
   )
+  (wire (pts (xy 74.93 153.67) (xy 75.565 153.67))
+    (stroke (width 0) (type default) (color 0 0 0 0))
+  )
   (wire (pts (xy 144.145 171.45) (xy 146.685 171.45))
     (stroke (width 0) (type default) (color 0 0 0 0))
@@
     (stroke (width 0) (type default) (color 0 0 0 0))
   )
+  (wire (pts (xy 59.69 151.13) (xy 80.01 151.13))
+    (stroke (width 0) (type default) (color 0 0 0 0))
+  )
   (wire (pts (xy 109.22 241.3) (xy 109.22 242.57))
-    (stroke (width 0) (type default) (color 0 0 0 0))
-  )
-  (wire (pts (xy 59.69 153.67) (xy 74.93 153.67))
     (stroke (width 0) (type default) (color 0 0 0 0))
   )
@@
   (symbol (lib_id "Device:R") (at 71.755 170.18 0) (unit 1)
     (in_bom yes) (on_board yes)
-    (property "Reference" "R4" (id 0) (at 73.787 171.45 90)
+    (property "Reference" "R3" (id 0) (at 73.787 171.45 90)
       (effects (font (size 1.27 1.27)) (justify left))
     )
@@
   (symbol (lib_id "Device:R") (at 59.055 251.46 90) (unit 1)
     (in_bom yes) (on_board yes)
-    (property "Reference" "R3" (id 0) (at 59.055 253.746 90))
+    (property "Reference" "R4" (id 0) (at 59.055 253.746 90))
     (property "Value" "5.1k" (id 1) (at 59.055 251.46 90))
     (property "Footprint" "Keyboard_Stuff:R_Axial_DIN0204_L3.6mm_D1.6mm_P5.08mm_Horizontal" (id 2) (at 59.055 253.238 90)
@@
   (symbol (lib_id "Device:R") (at 75.565 241.3 90) (unit 1)
     (in_bom yes) (on_board yes)
-    (property "Reference" "R5" (id 0) (at 75.565 239.268 90))
+    (property "Reference" "R7" (id 0) (at 75.565 239.268 90))
     (property "Value" "75" (id 1) (at 75.565 241.3 90))
     (property "Footprint" "Resistor_THT:R_Axial_DIN0204_L3.6mm_D1.6mm_P5.08mm_Horizontal" (id 2) (at 75.565 243.078 90)
@@
   (symbol (lib_id "Device:R") (at 130.81 207.645 270) (unit 1)
     (in_bom yes) (on_board yes)
-    (property "Reference" "R7" (id 0) (at 130.81 209.677 90))
+    (property "Reference" "R1" (id 0) (at 130.81 209.677 90))
     (property "Value" "1.5k" (id 1) (at 130.81 207.645 90))
     (property "Footprint" "Keyboard_Stuff:R_Axial_DIN0204_L3.6mm_D1.6mm_P5.08mm_Horizontal" (id 2) (at 130.81 205.867 90)
@@
   (symbol (lib_id "Device:R") (at 55.88 237.49 0) (unit 1)
     (in_bom yes) (on_board yes)
-    (property "Reference" "R1" (id 0) (at 57.912 238.76 90)
+    (property "Reference" "R5" (id 0) (at 57.912 238.76 90)
       (effects (font (size 1.27 1.27)) (justify left))
     )
@@
       (reference "Power1") (unit 1) (value "POWERLED") (footprint "Keyboard_Stuff:LED_D3.0mm")
     )
-    (path "/eaf0749f-fc67-4f3c-9a2d-cfa1273640a6"
-      (reference "R1") (unit 1) (value "1.5K") (footprint "Keyboard Stuff:R_Axial_DIN0204_L3.6mm_D1.6mm_P5.08mm_Horizontal")
+    (path "/9cb36fd3-6e1e-4c8b-8d0c-9f85fa199d85"
+      (reference "R1") (unit 1) (value "1.5k") (footprint "Keyboard_Stuff:R_Axial_DIN0204_L3.6mm_D1.6mm_P5.08mm_Horizontal")
     )
     (path "/11f288bc-9267-430d-973b-25fbc597cc5b"
       (reference "R2") (unit 1) (value "5.1k") (footprint "Keyboard_Stuff:R_Axial_DIN0204_L3.6mm_D1.6mm_P5.08mm_Horizontal")
     )
+    (path "/51d88d34-e7c1-4ff4-9140-56d9a685a6a7"
+      (reference "R3") (unit 1) (value "10K") (footprint "Keyboard_Stuff:R_Axial_DIN0204_L3.6mm_D1.6mm_P5.08mm_Horizontal")
+    )
     (path "/56edc18c-8dd5-4abf-81b5-9c7633852e22"
-      (reference "R3") (unit 1) (value "5.1k") (footprint "Keyboard_Stuff:R_Axial_DIN0204_L3.6mm_D1.6mm_P5.08mm_Horizontal")
-    )
-    (path "/51d88d34-e7c1-4ff4-9140-56d9a685a6a7"
-      (reference "R4") (unit 1) (value "10K") (footprint "Keyboard_Stuff:R_Axial_DIN0204_L3.6mm_D1.6mm_P5.08mm_Horizontal")
-    )
-    (path "/57bad49c-905f-40a3-be53-94667e4f70e0"
-      (reference "R5") (unit 1) (value "75") (footprint "Resistor_THT:R_Axial_DIN0204_L3.6mm_D1.6mm_P5.08mm_Horizontal")
+      (reference "R4") (unit 1) (value "5.1k") (footprint "Keyboard_Stuff:R_Axial_DIN0204_L3.6mm_D1.6mm_P5.08mm_Horizontal")
+    )
+    (path "/eaf0749f-fc67-4f3c-9a2d-cfa1273640a6"
+      (reference "R5") (unit 1) (value "1.5K") (footprint "Keyboard Stuff:R_Axial_DIN0204_L3.6mm_D1.6mm_P5.08mm_Horizontal")
     )
     (path "/b0f0c3ca-2cd9-4ee8-b4ec-3d8edf3e8fb1"
       (reference "R6") (unit 1) (value "75") (footprint "Keyboard_Stuff:R_Axial_DIN0204_L3.6mm_D1.6mm_P5.08mm_Horizontal")
     )
-    (path "/9cb36fd3-6e1e-4c8b-8d0c-9f85fa199d85"
-      (reference "R7") (unit 1) (value "1.5k") (footprint "Keyboard_Stuff:R_Axial_DIN0204_L3.6mm_D1.6mm_P5.08mm_Horizontal")
+    (path "/57bad49c-905f-40a3-be53-94667e4f70e0"
+      (reference "R7") (unit 1) (value "75") (footprint "Resistor_THT:R_Axial_DIN0204_L3.6mm_D1.6mm_P5.08mm_Horizontal")
     )
     (path "/6d8c26be-6a42-402b-acee-7b1a9d70afbd"
